File: hardware/msr20-c/msr20-c.kicad_pcb (KiCad board)
At the start: 2 copper layers, 73 parts, among them J1 TO ENCODER, J2 AUDIO OUT, J3 TO OLED, J4 SWD, J5 Conn_Coaxial, Q1 2N2907, Q2 2N2222, Q3 NPN, Q4 NPN, Q5 2N3904, Q6 2N3904, U1 Pico, U10 NCP1117-12_SOT223, U2 RF-BPF, U3 ADE-1+, U4 LTC455-FU, U5 AD7478, U6 74LS163, U7 CD74HC4046, U8 NCP1117-3.3_SOT223, U9 NCP1117-5.0_SOT223

Commit message: finish pcb rev 1, new png render
Parts:
- removed C22, C23: 1u, Capacitor_SMD:C_0805_2012Metric
- removed U10: NCP1117-12_SOT223, Package_TO_SOT_SMD:SOT-223-3_TabPin2
- added H1: MountingHole_Pad, MountingHole:MountingHole_3.2mm_M3_DIN965_Pad_TopBottom, F.Cu at (40.6, 22.9)
- added H2: MountingHole_Pad, MountingHole:MountingHole_3.2mm_M3_DIN965_Pad_TopBottom, F.Cu at (134.6, 22.9)
- added H3: MountingHole_Pad, MountingHole:MountingHole_3.2mm_M3_DIN965_Pad_TopBottom, F.Cu at (40.6, 113.0)
- added H4: MountingHole_Pad, MountingHole:MountingHole_3.2mm_M3_DIN965_Pad_TopBottom, F.Cu at (134.6, 113.0)
- added TP2: TestPoint, TestPoint:TestPoint_Pad_D1.0mm, F.Cu at (87.0, 53.3)
- added TP3: TestPoint, TestPoint:TestPoint_Pad_D1.0mm, F.Cu at (118.7, 66.0)
- added TP4: TestPoint, TestPoint:TestPoint_Pad_D1.0mm, F.Cu at (118.7, 59.7)
- added TP5: TestPoint, TestPoint:TestPoint_Pad_D1.0mm, F.Cu at (104.8, 83.2)
- added TP6: TestPoint, TestPoint:TestPoint_Pad_D1.0mm, F.Cu at (59.7, 52.1)
- RV1: footprint Resistor_SMD:R_0805_2012Metric -> Connector_PinHeader_2.54mm:PinHeader_1x03_P2.54mm_Vertical
- moved U3 171.8 mm to (84.5, 62.2), turned to 90 degrees
- moved JP1 166.9 mm to (59.7, 76.2)
- moved L2 158.6 mm to (95.2, 67.3)
- moved L3 154.0 mm to (100.3, 67.3)
- moved U4 151.8 mm to (97.8, 58.4)
- moved R19 151.4 mm to (101.0, 85.1), turned to 180 degrees
- moved U1 147.0 mm to (63.5, 92.1), turned to 90 degrees
- moved R16 147.0 mm to (101.0, 81.3)
- moved C5 145.7 mm to (87.0, 71.1)
- moved U5 142.7 mm to (95.9, 83.2), turned to 180 degrees
- moved C19 141.5 mm to (128.9, 103.7), turned to -90 degrees
- moved L4 140.4 mm to (117.5, 57.1), turned to 180 degrees
- moved C21 139.7 mm to (128.9, 89.5), turned to -90 degrees
- moved R13 139.6 mm to (108.6, 68.6), turned to 180 degrees
- moved C18 138.2 mm to (132.7, 103.7), turned to -90 degrees
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Connections:
- U1 pad 24: ADC-SCL -> ADC-SCK
- U1 pad 31: unconnected-(U1-GPIO26_ADC0-Pad31)_0 -> PLL-IN
- U1 pad 9: PLL-IN -> unconnected-(U1-GPIO6-Pad9)
Routing:
- net +5V: track 0.00 -> 235.0 mm, vias 0 -> 5
- net +3.3V: track 0.00 -> 123.3 mm, vias 0 -> 3
- net Net-(J1-Pin_1): track 0.00 -> 83.1 mm
- net Net-(J1-Pin_2): track 0.00 -> 82.0 mm
- net GND: track 13.0 -> 81.6 mm, vias 0 -> 18
- net Net-(U3-RF): track 2.54 -> 66.2 mm
- net Net-(U1-GPIO22): track 0.00 -> 53.4 mm
- net Net-(U5-VIN): track 0.00 -> 47.8 mm
- net Net-(Q6-B): track 0.00 -> 43.6 mm
- net Net-(J3-Pin_1): track 0.00 -> 34.6 mm
- net /Phase-locked loop/OUT: track 0.00 -> 33.0 mm
- net Net-(J3-Pin_2): track 0.00 -> 31.0 mm
- net PLL-IN: track 0.00 -> 25.6 mm, vias 0 -> 1
- net VIN: track 0.00 -> 22.9 mm
- net Net-(Q3-B): track 0.00 -> 21.3 mm
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- added copper zone on B.Cu, net GND
Other:
- board outline added: 104.1 x 100.3 mm
- board text added: "ADC"
- board text added: "AUDIO OUT"
- board text added: "ENCODER"
- board text added: "IF AMP"
- board text added: "IF BPF"
- board text added: "IF VGA"
- board text added: "MSR-20 Cooper Union EE 2024 J. Yoon C. Van West E. Murphy J.W. Lee T. Coor"
- board text added: "Mixer"
- board text added: "OLED"
- board text added: "PANEL"
- board text added: "RF BPF"
- board text removed: "BPF"

Commit message: plot msr20-c schematic and pcb
Parts:
- moved C1 51.1 mm to (159.3, 110.5)
- moved C10 51.1 mm to (157.4, 97.8)
- moved C11 51.1 mm to (153.0, 97.8)
- moved C12 51.1 mm to (177.1, 98.4)
- moved C13 51.1 mm to (104.1, 81.3)
- moved C14 51.1 mm to (104.1, 85.1)
- moved C18 51.1 mm to (177.1, 129.1)
- moved C19 51.1 mm to (173.3, 129.1)
- moved C2 51.1 mm to (119.3, 58.4)
- moved C20 51.1 mm to (177.1, 114.9)
- moved C21 51.1 mm to (173.3, 114.9)
- moved C3 51.1 mm to (119.3, 62.2)
- moved C4 51.1 mm to (102.8, 67.3)
- moved C6 51.1 mm to (153.0, 90.2)
- moved C7 51.1 mm to (161.9, 78.7)
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Other:
- outline, holes or cut-outs redrawn
- board text added: "MSR-20 REV. 1 Cooper Union EE 2024 J. Yoon C. Van West E. Murphy J.W. Lee T. Coor"
- board text removed: "MSR-20 Cooper Union EE 2024 J. Yoon C. Van West E. Murphy J.W. Lee T. Coor"
