File: hardware/msr20-c/msr20-c.kicad_sch (KiCad schematic)
At the start: 14 parts, among them J1 TO ENCODER, J2 AUDIO OUT, J3 TO OLED, J4 SWD, U1 Pico

Commit message: plot msr20-c schematic and pcb
Other:
- title: (none) -> MSR-20
Changed lines of the file:
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@@
 	(paper "USLetter")
 	(title_block
-		(date "2024-04-20")
+		(title "MSR-20")
+		(date "2024-04-29")
 		(rev "1")
 	)
