File: hardware/msr20-c/power.kicad_sch (KiCad schematic)
At the start: 9 parts, among them U10 NCP1117-12_SOT223, U8 NCP1117-3.3_SOT223, U9 NCP1117-5.0_SOT223

Commit message: finish pcb rev 1, new png render
Parts:
- removed C22, C23: 1u, Capacitor_SMD:C_0805_2012Metric, symbol Device:C
- removed U10: NCP1117-12_SOT223, Package_TO_SOT_SMD:SOT-223-3_TabPin2, symbol Regulator_Linear:NCP1117-12_SOT223
