File: hardware/msr20-c/rf.kicad_sch (KiCad schematic)
At the start: 14 parts, among them J5 Conn_Coaxial, Q1 2N2907, Q2 2N2222, U2 RF-BPF, U3 ADE-1+

Commit message: pcb: pll, lna, rf-bpf layout
Parts:
- J5: footprint Connector_Coaxial:BNC_Amphenol_031-5539_Vertical -> Connector_Coaxial:BNC_TEConnectivity_1478035_Horizontal
Changed lines of the file:
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@@
 			)
 		)
-		(property "Footprint" "Connector_Coaxial:BNC_Amphenol_031-5539_Vertical"
+		(property "Footprint" "Connector_Coaxial:BNC_TEConnectivity_1478035_Horizontal"
 			(at 44.45 85.09 0)
 			(effects

Commit message: finish pcb rev 1, new png render
Parts:
- added TP2: TestPoint, TestPoint:TestPoint_Pad_D1.0mm, symbol Connector:TestPoint
Connections:
- net at U2.7 (OUT), U2.8 (OUT), U3.3 (RF): now also TP2.1
Changed lines of the file:
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@@
+	)
+	(junction
+		(at 160.02 77.47)
+		(diameter 0)
+		(color 0 0 0 0)
 	)
 	(junction
@@
 	(wire
 		(pts
-			(xy 144.78 77.47) (xy 176.53 77.47)
+			(xy 144.78 77.47) (xy 160.02 77.47)
 		)
 		(stroke
@@
 		(pts
 			(xy 77.47 77.47) (xy 77.47 80.01)
+		)
+		(stroke
+			(width 0)
+			(type default)
+		)
+	)
+	(wire
+		(pts
+			(xy 160.02 77.47) (xy 160.02 81.28)
+		)
+		(stroke
+			(width 0)
+			(type default)
+		)
+	)
+	(wire
+		(pts
+			(xy 160.02 77.47) (xy 176.53 77.47)
 		)
 		(stroke
@@
 					(unit 1)
 				)
+			)
+		)
+	)
+	(symbol
+		(lib_id "Connector:TestPoint")
+		(at 160.02 81.28 180)
+		(unit 1)
+		(exclude_from_sim no)
+		(in_bom yes)
+		(on_board yes)
+		(dnp no)
+		(property "Reference" "TP2"
+			(at 155.956 87.63 0)
+			(effects
+				(font
+					(size 1.27 1.27)
+				)
+				(justify right)
+			)
+		)
+		(property "Value" "TestPoint"
+			(at 155.956 90.17 0)
+			(effects
+				(font
+					(size 1.27 1.27)
+				)
+				(justify right)
+			)
+		)
+		(property "Footprint" "TestPoint:TestPoint_Pad_D1.0mm"
+			(at 154.94 81.28 0)
+			(effects
+				(font
+					(size 1.27 1.27)
+				)
+				(hide yes)
+			)
+		)
+		(property "Datasheet" "~"
+			(at 154.94 81.28 0)
+			(effects
+				(font
+					(size 1.27 1.27)
+				)
+				(hide yes)
+			)
+		)
+		(property "Description" "test point"
+			(at 160.02 81.28 0)
+			(effects
+				(font
+					(size 1.27 1.27)
+				)
+				(hide yes)
+			)
+		)
+		(pin "1"
+		)
+		(instances
+			(project "msr20-c"
+				(path "/3d24e86e-b070-4f0e-8c28-04e9dd9d95d1/c9c41028-bd5c-45d5-9f40-d2ea8ca6f8e9"
+					(reference "TP2")
+					(unit 1)
+				)

Commit message: plot msr20-c schematic and pcb
Other:
- title: (none) -> RF Stage
Changed lines of the file:
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@@
 	(generator "eeschema")
 	(generator_version "8.0")
-	(paper "A4")
+	(paper "USLetter")
+	(title_block
+		(title "RF Stage")
+		(date "2024-04-29")
+		(rev "1")
+	)
 	(junction
 		(at 109.22 87.63)
@@
 	(text "Low-Noise Amplifier"
 		(exclude_from_sim no)
-		(at 38.1 24.13 0)
+		(at 25.4 24.13 0)
 		(effects
 			(font
